File: pcb/multisensor/multisensor.kicad_pcb (KiCad board)
At the start: 2 copper layers, 50 x 40 mm, 29 parts, among them J1 TTL, J2 mmWave_Data, J3 mmWave_Support, J4 PIR_Sensor, J5 BME680, J6 BH1750, J7 10118193-0001LF, Q1 PN2222A, Q2 PN2222A, SW1 RESET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

Commit message: update gerber files
Parts:
- moved REF** 0.71 mm to (131.9, 119.9)
- moved REF** 0.71 mm to (174.9, 119.9)
- moved REF** 0.50 mm to (131.9, 91.4)
- moved REF** 0.50 mm to (174.9, 91.4)
- moved SW1 0.38 mm to (164.8, 111.0)
Changed lines of the file:
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@@
       (drillshape 0)
       (scaleselection 1)
-      (outputdirectory "plots/")
+      (outputdirectory "manufacturing/gerber")
     )
   )
@@
   )
   (footprint "MountingHole:MountingHole_2.7mm_Pad" (layer "F.Cu")
-    (at 131.375 120.375)
+    (at 131.875 119.875)
     (descr "Mounting Hole 2.7mm")
     (tags "mounting hole 2.7mm")
@@
   )
   (footprint "MountingHole:MountingHole_2.7mm_Pad" (layer "F.Cu")
-    (at 131.375 91.375)
+    (at 131.875 91.375)
     (descr "Mounting Hole 2.7mm")
     (tags "mounting hole 2.7mm")
@@
   )
   (footprint "MountingHole:MountingHole_2.7mm_Pad" (layer "F.Cu")
-    (at 175.375 120.375)
+    (at 174.875 119.875)
     (descr "Mounting Hole 2.7mm")
     (tags "mounting hole 2.7mm")
@@
   )
   (footprint "MountingHole:MountingHole_2.7mm_Pad" (layer "F.Cu")
-    (at 175.375 91.375)
+    (at 174.875 91.375)
     (descr "Mounting Hole 2.7mm")
     (tags "mounting hole 2.7mm")
@@
   )
   (footprint "Button_Switch_THT:SW_PUSH_6mm" (layer "F.Cu")
-    (at 165.125 111.125)
+    (at 164.775 110.975)
     (descr "https://www.omron.com/ecb/products/pdf/en-b3f.pdf")
     (tags "tact sw push 6mm")
@@
   (via (at 153.375 103.875) (size 0.8) (drill 0.4) (layers "F.Cu" "B.Cu") (free) (net 11))
   (via (at 135.5625 109.8625) (size 0.8) (drill 0.4) (layers "F.Cu" "B.Cu") (free) (net 11))
-  (via (at 168.375 112.075) (size 0.8) (drill 0.4) (layers "F.Cu" "B.Cu") (free) (net 11))
+  (via (at 167.975 111.975) (size 0.8) (drill 0.4) (layers "F.Cu" "B.Cu") (free) (net 11))
   (via (at 135.1625 96.7625) (size 0.8) (drill 0.4) (layers "F.Cu" "B.Cu") (free) (net 11))
   (via (at 131.6625 113.8625) (size 0.8) (drill 0.4) (layers "F.Cu" "B.Cu") (free) (net 11))
@@
   (via (at 153.375 91.375) (size 0.8) (drill 0.4) (layers "F.Cu" "B.Cu") (free) (net 11))
   (via (at 171.5625 88.675) (size 0.8) (drill 0.4) (layers "F.Cu" "B.Cu") (free) (net 11))
-  (segment (start 147.480698 100.393198) (end 148.348896 99.525) (width 0.25) (layer "F.Cu") (net 13))
-  (segment (start 147.2375 101.9) (end 147.480698 101.656802) (width 0.25) (layer "F.Cu") (net 13))
-  (segment (start 144.2 101.70962) (end 144.39038 101.9) (width 0.25) (layer "F.Cu") (net 13))
-  (segment (start 160.3625 106.175) (end 166.01 106.175) (width 0.25) (layer "F.Cu") (net 13))
-  (segment (start 144.2 99.4) (end 144.2 101.70962) (width 0.25) (layer "F.Cu") (net 13))
   (segment (start 145.775 99.075) (end 144.525 99.075) (width 0.25) (layer "F.Cu") (net 13))
   (segment (start 144.39038 101.9) (end 147.2375 101.9) (width 0.25) (layer "F.Cu") (net 13))
-  (segment (start 157.5625 99.525) (end 157.5625 103.375) (width 0.25) (layer "F.Cu") (net 13))
+  (segment (start 144.2 101.70962) (end 144.39038 101.9) (width 0.25) (layer "F.Cu") (net 13))
+  (segment (start 166.01 106.175) (end 166.075 106.24) (width 0.25) (layer "F.Cu") (net 13))
   (segment (start 144.525 99.075) (end 144.2 99.4) (width 0.25) (layer "F.Cu") (net 13))
+  (segment (start 160.3625 106.175) (end 166.01 106.175) (width 0.25) (layer "F.Cu") (net 13))
+  (segment (start 147.2375 101.9) (end 147.480698 101.656802) (width 0.25) (layer "F.Cu") (net 13))
+  (segment (start 144.2 99.4) (end 144.2 101.70962) (width 0.25) (layer "F.Cu") (net 13))
+  (segment (start 147.480698 100.393198) (end 148.348896 99.525) (width 0.25) (layer "F.Cu") (net 13))
+  (segment (start 157.5625 99.9625) (end 157.5625 103.375) (width 0.25) (layer "F.Cu") (net 13))
+  (segment (start 157.125 99.525) (end 157.5625 99.9625) (width 0.25) (layer "F.Cu") (net 13))
   (segment (start 157.5625 103.375) (end 160.3625 106.175) (width 0.25) (layer "F.Cu") (net 13))
-  (segment (start 148.348896 99.525) (end 157.5625 99.525) (width 0.25) (layer "F.Cu") (net 13))
-  (segment (start 166.01 106.175) (end 166.075 106.24) (width 0.25) (layer "F.Cu") (net 13))
   (segment (start 147.480698 101.656802) (end 147.480698 100.393198) (width 0.25) (layer "F.Cu") (net 13))
+  (segment (start 148.348896 99.525) (end 157.125 99.525) (width 0.25) (layer "F.Cu") (net 13))
   (segment (start 143.275 97.075) (end 145.775 97.075) (width 0.25) (layer "F.Cu") (net 14))
   (via (at 143.275 97.075) (size 0.8) (drill 0.4) (layers "F.Cu" "B.Cu") (free) (net 14))
@@
   (segment (start 171.5625 90.175) (end 171.5625 97.675) (width 0.25) (layer "B.Cu") (net 26))
   (segment (start 143.275 89.075) (end 145.775 89.075) (width 0.25) (layer "F.Cu") (net 31))
-  (segment (start 165.125 111.125) (end 160.88375 106.88375) (width 0.25) (layer "F.Cu") (net 31))
+  (segment (start 164.775 110.775) (end 160.88375 106.88375) (width 0.25) (layer "F.Cu") (net 31))
   (segment (start 160.88375 106.88375) (end 160.475 106.88375) (width 0.25) (layer "F.Cu") (net 31))
+  (segment (start 164.775 110.975) (end 171.275 110.975) (width 0.25) (layer "F.Cu") (net 31))
   (segment (start 141.6875 89.075) (end 143.275 89.075) (width 0.25) (layer "F.Cu") (net 31))
-  (segment (start 165.125 111.125) (end 171.625 111.125) (width 0.25) (layer "F.Cu") (net 31))
+  (segment (start 164.775 110.975) (end 164.775 110.775) (width 0.25) (layer "F.Cu") (net 31))
   (via (at 143.275 89.075) (size 0.8) (drill 0.4) (layers "F.Cu" "B.Cu") (net 31))
-  (segment (start 139.388604 94.165) (end 138.058604 95.495) (width 0.25) (layer "B.Cu") (net 31))
-  (segment (start 129.755 95.495) (end 129.005 96.245) (width 0.25) (layer "B.Cu") (net 31))
-  (segment (start 143.275 89.075) (end 143.275 93.495) (width 0.25) (layer "B.Cu") (net 31))
+  (segment (start 159.405 116.845) (end 164.775 111.475) (width 0.25) (layer "B.Cu") (net 31))
   (segment (start 129.005 96.245) (end 129.005 110.585) (width 0.25) (layer "B.Cu") (net 31))
   (segment (start 143.275 93.495) (end 142.605 94.165) (width 0.25) (layer "B.Cu") (net 31))
+  (segment (start 138.058604 95.495) (end 129.755 95.495) (width 0.25) (layer "B.Cu") (net 31))
+  (segment (start 130.255 111.835) (end 138.878604 111.835) (width 0.25) (layer "B.Cu") (net 31))
+  (segment (start 143.275 89.075) (end 143.275 93.495) (width 0.25) (layer "B.Cu") (net 31))
+  (segment (start 142.605 94.165) (end 139.388604 94.165) (width 0.25) (layer "B.Cu") (net 31))
+  (segment (start 139.388604 94.165) (end 138.058604 95.495) (width 0.25) (layer "B.Cu") (net 31))
+  (segment (start 129.005 110.585) (end 130.255 111.835) (width 0.25) (layer "B.Cu") (net 31))
   (segment (start 138.878604 111.835) (end 143.888604 116.845) (width 0.25) (layer "B.Cu") (net 31))
-  (segment (start 130.255 111.835) (end 138.878604 111.835) (width 0.25) (layer "B.Cu") (net 31))
-  (segment (start 138.058604 95.495) (end 129.755 95.495) (width 0.25) (layer "B.Cu") (net 31))
-  (segment (start 129.005 110.585) (end 130.255 111.835) (width 0.25) (layer "B.Cu") (net 31))
-  (segment (start 159.405 116.845) (end 165.125 111.125) (width 0.25) (layer "B.Cu") (net 31))
+  (segment (start 129.755 95.495) (end 129.005 96.245) (width 0.25) (layer "B.Cu") (net 31))
   (segment (start 143.888604 116.845) (end 159.405 116.845) (width 0.25) (layer "B.Cu") (net 31))
-  (segment (start 142.605 94.165) (end 139.388604 94.165) (width 0.25) (layer "B.Cu") (net 31))
+  (segment (start 164.775 111.475) (end 164.775 110.975) (width 0.25) (layer "B.Cu") (net 31))
   (segment (start 160.975 97.075) (end 163.475 97.075) (width 0.25) (layer "F.Cu") (net 32))
   (segment (start 163.475 97.075) (end 163.765 97.365) (width 0.25) (layer "F.Cu") (net 32))
