File: pcb/multisensor/multisensor.kicad_pcb (KiCad board)
At the start: 2 copper layers, 50 x 40 mm, 29 parts, among them J1 TTL, J2 mmWave_Data, J3 mmWave_Support, J4 PIR_Sensor, J5 BME680, J6 BH1750, J7 10118193-0001LF, Q1 PN2222A, Q2 PN2222A, SW1 RESET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

Commit message: fix pcb layout
Parts:
- J1: value TTL -> TTL_Serial
- U1: moved to B.Cu
- moved R5 22.7 mm to (147.4, 97.6), turned to -90 degrees
- moved C1 21.8 mm to (160.8, 120.5), turned to 0 degrees
- moved C2 21.8 mm to (160.8, 117.9), turned to 0 degrees
- moved U2 21.8 mm to (160.8, 114.4), turned to 0 degrees
- moved C3 21.8 mm to (160.8, 110.9)
- moved C4 21.8 mm to (160.8, 108.3)
- moved R6 18.5 mm to (151.4, 97.6), turned to 90 degrees
- moved R3 17.5 mm to (157.4, 91.2), turned to 90 degrees
- moved C5 15.9 mm to (153.4, 91.2), turned to -90 degrees
- moved SW1 15.3 mm to (150.1, 106.6)
- moved R7 14.7 mm to (155.4, 97.6), turned to 90 degrees
- moved J5 13.3 mm to (135.4, 109.8)
- moved J2 12.6 mm to (166.1, 106.2), turned to 0 degrees
- moved R8 11.4 mm to (159.4, 97.6), turned to 90 degrees
- moved J1 9.58 mm to (146.6, 120.3), turned to 180 degrees
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Connections:
- Q1 pad 1: RTS -> Net-(Q1-B)
- Q1 pad 2: Net-(Q1-B) -> RTS
- Q2 pad 1: DTR -> Net-(Q2-B)
- Q2 pad 2: Net-(Q2-B) -> DTR
Routing:
- net +3.3V: track 102.1 -> 48.3 mm
- net nRST: track 92.0 -> 52.8 mm
- net +5V: track 111.4 -> 72.5 mm, vias 2 -> 0
- net GPIO0: track 45.7 -> 19.8 mm, vias 2 -> 1
- net DTR: track 7.82 -> 32.0 mm
- net MMW_TX: track 32.5 -> 8.96 mm
- net MMW_RX: track 24.3 -> 7.58 mm
- net RX: track 49.3 -> 33.7 mm
- net SDA: track 56.2 -> 70.5 mm, vias 1 -> 2
- net SCL: track 62.8 -> 77.1 mm, vias 1 -> 2
- net TX: track 47.2 -> 36.7 mm
- net Net-(U1-EN): track 8.55 -> 14.5 mm, vias 0 -> 1
- net MMW_IO2: track 23.3 -> 18.3 mm
- net RTS: track 12.0 -> 16.6 mm
- net GND: track 5.80 -> 1.99 mm
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Other:
- board size 50 x 40 mm -> 40 x 40 mm
- board text added: "IO2"
- board text added: "PIR"

Commit message: finalize v0.2.0
Parts:
- added G***: LOGO, *Multisensor:logo, F.Cu at (160.2, 85.7)
